File: PCB/WorldEdit-HackPad.kicad_pcb (KiCad board)
At the start: 2 copper layers, 85.7 x 85.7 mm, 31 parts, among them SW1 SW_Push, SW10 SW_Push, SW11 SW_Push, SW12 SW_Push, SW13 SW_Push, SW14 SW_Push, SW15 SW_Push, SW2 SW_Push, SW3 SW_Push, SW4 SW_Push, SW5 SW_Push, SW6 SW_Push, SW7 SW_Push, SW8 SW_Push, SW9 SW_Push, U1 XIAO-RP2040-DIP

Commit message: Update Schem and PCB
Parts:
- moved D11 5.32 mm to (50.0, 81.0)
- moved D12 5.32 mm to (69.1, 81.0)
- moved D15 5.32 mm to (92.9, 81.0)
- moved D14 5.32 mm to (92.9, 61.9)
- moved D2 5.32 mm to (50.0, 19.1)
- moved D3 5.32 mm to (69.7, 19.1)
- moved D5 5.32 mm to (50.0, 38.1)
- moved D6 5.32 mm to (69.1, 38.1)
- moved D8 5.32 mm to (50.0, 57.1)
- moved D9 5.32 mm to (69.1, 57.1)
- moved SW1 5.32 mm to (33.5, 23.5)
- moved SW10 5.32 mm to (71.6, 42.5)
- moved SW11 5.32 mm to (71.6, 61.6)
- moved SW14 5.32 mm to (95.4, 66.4)
- moved SW2 5.32 mm to (33.5, 42.5)
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Connections:
- SW1 pad 2: Net-(U1-GPIO3/MOSI) -> Net-(U1-GPIO2/SCK)
- SW10 pad 2: Net-(U1-GPIO2/SCK) -> Net-(U1-GPIO1/RX)
- SW11 pad 2: Net-(U1-GPIO2/SCK) -> Net-(U1-GPIO4/MISO)
- SW12 pad 2: Net-(U1-GPIO2/SCK) -> Net-(U1-GPIO3/MOSI)
- SW14 pad 2: Net-(U1-GPIO1/RX) -> Net-(U1-GPIO4/MISO)
- SW15 pad 2: Net-(U1-GPIO1/RX) -> Net-(U1-GPIO3/MOSI)
- SW2 pad 2: Net-(U1-GPIO3/MOSI) -> Net-(U1-GPIO1/RX)
- SW3 pad 2: Net-(U1-GPIO3/MOSI) -> Net-(U1-GPIO4/MISO)
- SW5 pad 2: Net-(U1-GPIO4/MISO) -> Net-(U1-GPIO2/SCK)
- SW6 pad 2: Net-(U1-GPIO4/MISO) -> Net-(U1-GPIO1/RX)
- SW8 pad 2: Net-(U1-GPIO4/MISO) -> Net-(U1-GPIO3/MOSI)
Routing:
- net Net-(U1-GPIO4/MISO): track 171.5 -> 108.5 mm, vias 2 -> 0
- net Net-(U1-GPIO2/SCK): track 106.9 -> 75.9 mm, vias 2 -> 0
- net Net-(U1-GPIO1/RX): track 64.9 -> 84.3 mm, vias 2 -> 0
- net Net-(U1-GPIO0/TX): track 70.1 -> 54.8 mm, vias 2 -> 0
- net Net-(D3-DOUT): track 48.6 -> 62.3 mm
- net +5V: track 350.2 -> 337.2 mm, vias 6 -> 2
- net GND: track 351.4 -> 340.1 mm, vias 3 -> 11
- net Net-(U1-GPIO3/MOSI): track 145.6 -> 139.7 mm, vias 3 -> 0
- net Net-(D7-DOUT): track 25.3 -> 31.0 mm, vias 2 -> 4
- net Net-(U1-GPIO29/ADC3/A3): track 122.6 -> 116.9 mm, vias 4 -> 0
- net Net-(U1-GPIO6/SDA): track 104.5 -> 99.0 mm, vias 2 -> 0
- net Net-(D4-DOUT): track 30.1 -> 24.8 mm, vias 2 -> 4
- net Net-(D6-DOUT): track 54.2 -> 58.9 mm, vias 2 -> 4
- net Net-(D8-DOUT): track 24.5 -> 28.5 mm
- net Net-(D2-DOUT): track 26.9 -> 23.9 mm
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