File: PCB/WorldEdit-HackPad.kicad_sch (KiCad schematic)
At the start: 31 parts, among them SW1 SW_Push, SW10 SW_Push, SW11 SW_Push, SW12 SW_Push, SW13 SW_Push, SW14 SW_Push, SW15 SW_Push, SW2 SW_Push, SW3 SW_Push, SW4 SW_Push, SW5 SW_Push, SW6 SW_Push, SW7 SW_Push, SW8 SW_Push, SW9 SW_Push, U1 XIAO-RP2040-DIP

Commit message: Update Schem and PCB
Connections:
- net at SW13.2, U1.8 (GPIO1/RX): now also SW10.2, SW2.2, SW6.2; no longer SW14.2, SW15.2
- new net: SW12.2, SW15.2, SW4.2, SW8.2, U1.11 (GPIO3/MOSI)
- new net: SW11.2, SW14.2, SW3.2, SW7.2, U1.10 (GPIO4/MISO)
- new net: SW1.2, SW5.2, SW9.2, U1.9 (GPIO2/SCK)
